File: Raspberry/Raspberry.sch (KiCad schematic (older format))
At the start: 28 parts, among them J2 Conn_01x02, J3 Conn_01x03, J4 Conn_01x03, J5 Conn_01x03, J81 J8Header, J82 J8Header, Q1 BC337, Q2 BC337

Commit message: Korrekturen
Parts:
- added W3: Wire, RasperryLib:Wire_long, symbol Wire
- J4, J5: footprint RasperryLib:Conn_Small1x3 -> RasperryLib:Connector1x3
Connections:
- wire segments 184 -> 187

Commit message: Buzzer 5v
Parts:
- removed RL1: Relais, RasperryLib:Relais, symbol Relais-RESCUE-Raspberry
- added RL1: Relais, RasperryLib:Relais, symbol Relais
Connections:
- wire segments 187 -> 188
Changed lines of the file:
@@
-$EndComp
-$Comp
-L Relais-RESCUE-Raspberry RL1
-U 1 1 5B956127
-P 11100 5350
-F 0 "RL1" H 10650 4300 60  0000 C CNN
-F 1 "Relais" H 10600 5350 60  0000 C CNN
-F 2 "RasperryLib:Relais" H 11100 5350 60  0001 C CNN
-F 3 "" H 11100 5350 60  0001 C CNN
-	1    11100 5350
-	0    1    1    0
 $EndComp
 $Comp
@@
 	1    0    0    -1
 $EndComp
+$Comp
+L Relais RL1
+U 1 1 5BD373A7
+P 10600 4900
+F 0 "RL1" H 10600 4350 60  0000 C CNN
+F 1 "Relais" H 10550 5400 60  0000 C CNN
+F 2 "RasperryLib:Relais" H 11050 5400 60  0001 C CNN
+F 3 "" H 11050 5400 60  0001 C CNN
+	1    10600 4900
+	0    1    1    0
+$EndComp
 Wire Wire Line
 	3800 1300 3950 1300
@@
 Connection ~ 10250 4100
 Wire Wire Line
-	6350 5200 9850 5200
-Wire Wire Line
-	6350 5200 6350 5550
-Wire Wire Line
 	6350 5950 6350 6150
 Wire Wire Line
@@
 	4700 2900 4700 2200
 Wire Wire Line
-	4000 2200 4700 2200
-Wire Wire Line
-	4000 1300 4000 2200
+	4700 2200 4000 2200
+Wire Wire Line
+	4000 2200 4000 1300
 Wire Wire Line
 	4000 1300 4050 1300
@@
 	10700 2500 10300 2500
 Wire Wire Line
-	10300 3200 10300 2500
-Wire Wire Line
-	4700 3200 10300 3200
+	10300 2500 10300 3200
+Wire Wire Line
+	10300 3200 4700 3200
 Wire Wire Line
 	7850 3450 7850 2200
@@
 	3700 3700 4650 3700
 Connection ~ 5300 3700
+Connection ~ 6350 3700
+Wire Wire Line
+	4650 3700 4650 3800
+Wire Wire Line
+	4650 3800 6350 3800
+Wire Wire Line
+	6350 3800 6350 5550
 $EndSCHEMATC
